File: finalPCB.kicad_pcb (KiCad board)
At the start: 2 copper layers, 110 x 110 mm, 44 parts, among them J2 FCR7350R, J3 FCR7350R, J4 FCR7350R, Q1 IRLML6401, Q2 IRLML6401, Q3 IRLML6401, Q4 IRLML6401, Q5 IRLML6401, SW1 SW_Omron_B3FS, SW2 SW_Omron_B3FS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

Commit message: Some routing done. There is still more schematic work to be done....
Parts:
- added C1: 100n, Capacitor_SMD:C_0805_2012Metric_Pad1.18x1.45mm_HandSolder, F.Cu at (154.5, 79.0)
- added C10: 10uF, Capacitor_SMD:C_0805_2012Metric_Pad1.18x1.45mm_HandSolder, F.Cu at (173.3, 111.3)
- added C11: 10uF, Capacitor_SMD:C_0805_2012Metric_Pad1.18x1.45mm_HandSolder, F.Cu at (161.4, 113.8)
- added C13: 0.22uF, Capacitor_SMD:C_0805_2012Metric_Pad1.18x1.45mm_HandSolder, F.Cu at (224.8, 76.8)
- added C14: 10uf, Capacitor_SMD:C_0805_2012Metric_Pad1.18x1.45mm_HandSolder, F.Cu at (224.8, 79.8)
- added C2: 330n, Capacitor_SMD:C_0805_2012Metric_Pad1.18x1.45mm_HandSolder, F.Cu at (173.5, 71.0)
- added C6: 10uF, Capacitor_SMD:C_0805_2012Metric_Pad1.18x1.45mm_HandSolder, F.Cu at (165.9, 100.8)
- added C7: 10uF, Capacitor_SMD:C_0805_2012Metric_Pad1.18x1.45mm_HandSolder, F.Cu at (172.9, 108.3)
- added C8: 10uF, Capacitor_SMD:C_0805_2012Metric_Pad1.18x1.45mm_HandSolder, F.Cu at (154.9, 122.8)
- added C9: 10uF, Capacitor_SMD:C_0805_2012Metric_Pad1.18x1.45mm_HandSolder, F.Cu at (173.4, 114.3)
- added D1: zener4.8, Diode_THT:D_A-405_P10.16mm_Horizontal, F.Cu at (142.9, 116.9)
- added D2: zener2.5, Diode_THT:D_A-405_P10.16mm_Horizontal, F.Cu at (160.0, 78.5)
- added J1: 9V Battery, Connector_PinSocket_2.54mm:PinSocket_1x02_P2.54mm_Vertical, F.Cu at (239.9, 49.2)
- added J5: Switch, Connector_PinSocket_2.54mm:PinSocket_1x02_P2.54mm_Vertical, F.Cu at (244.5, 49.2)
- added K1: HFD4/005, HFD4_005:HFD4_005, F.Cu at (187.4, 107.0)
- added K2: HFD4/005, HFD4_005:HFD4_005, F.Cu at (187.7, 123.0)
- added K3: HFD4/005, HFD4_005:HFD4_005, F.Cu at (152.2, 111.7)
- added Q6: NMOS, Package_TO_SOT_SMD:SOT-23-3, F.Cu at (160.8, 107.9)
- added R22: 15K, Resistor_SMD:R_0805_2012Metric_Pad1.20x1.40mm_HandSolder, F.Cu at (172.8, 104.8)
- added R23: 5K, Resistor_SMD:R_0805_2012Metric_Pad1.20x1.40mm_HandSolder, F.Cu at (165.9, 104.3)
- added R24: 10K, Resistor_SMD:R_0805_2012Metric_Pad1.20x1.40mm_HandSolder, F.Cu at (142.9, 120.3)
- added R25: 5K, Resistor_SMD:R_0805_2012Metric_Pad1.20x1.40mm_HandSolder, F.Cu at (150.9, 116.8)
- added R26: 15K, Resistor_SMD:R_0805_2012Metric_Pad1.20x1.40mm_HandSolder, F.Cu at (150.9, 120.3)
- added R27: 10K, Resistor_SMD:R_0805_2012Metric_Pad1.20x1.40mm_HandSolder, F.Cu at (170.4, 121.8)
- added R28: 30K, Resistor_SMD:R_0805_2012Metric_Pad1.20x1.40mm_HandSolder, F.Cu at (170.4, 118.3)
- added U1: 7414, Package_DIP:DIP-14_W7.62mm_LongPads, F.Cu at (165.9, 74.8)
- added U3: LMV358, Package_SO:SOIC-8_3.9x4.9mm_P1.27mm, F.Cu at (167.3, 111.3)
- added U4: LMV358, Package_SO:SOIC-8_3.9x4.9mm_P1.27mm, F.Cu at (161.8, 119.3)
- added U5: L7805, Package_TO_SOT_SMD:TO-263-3_TabPin2, F.Cu at (186.2, 58.0)
- moved R30 47.4 mm to (139.1, 74.0)
- moved R5 47.4 mm to (139.1, 71.0)
- moved R3 32.0 mm to (151.0, 75.0), turned to -90 degrees
- moved R4 31.3 mm to (160.0, 72.6), turned to 90 degrees
- moved R1 30.9 mm to (151.0, 70.6), turned to -90 degrees
- moved R2 29.0 mm to (155.0, 72.5)
Connections:
- C12 pad 1: Net-(U3B-+) -> CURRENT
- R29 pad 2: Net-(U3B-+) -> CURRENT
Routing:
- net +5V: track 0.00 -> 44.9 mm, vias 0 -> 1
- net HighRange: track 0.00 -> 38.5 mm, vias 0 -> 3
- net LowRange: track 0.00 -> 25.8 mm
- net VRf: track 0.00 -> 25.7 mm
- net Net-(U3A-+): track 0.00 -> 13.2 mm
- net Net-(U4A--): track 0.00 -> 12.8 mm
- net Net-(D1-K): track 0.00 -> 9.45 mm
- net RangeSel: track 0.00 -> 9.31 mm
- net Net-(U4B--): track 0.00 -> 8.57 mm
- net Net-(K3--): track 0.00 -> 3.90 mm

Commit message: V0.1 Done
The first full routing is complete. There is no LM35 sensor included.

PS.
The silkscreen art can be removed, but please no;)
Parts:
- added Q7: NMOS, Package_TO_SOT_SMD:SOT-23-3, F.Cu at (179.5, 119.0)
- added Q8: NMOS, Package_TO_SOT_SMD:SOT-23-3, F.Cu at (179.0, 103.0)
- moved Q5 77.5 mm to (106.0, 56.0)
- moved R21 74.5 mm to (110.5, 56.0)
- moved R20 74.4 mm to (101.4, 56.0), turned to -90 degrees
- moved R16 73.8 mm to (97.0, 60.0)
- moved R14 70.3 mm to (101.5, 66.0), turned to 90 degrees
- moved R19 70.1 mm to (96.9, 55.0)
- moved Q4 70.0 mm to (106.1, 61.0)
- moved R10 69.8 mm to (96.9, 70.0)
- moved R8 67.8 mm to (101.5, 76.0), turned to -90 degrees
- moved R18 67.2 mm to (110.5, 61.0)
- moved R17 66.3 mm to (101.5, 61.0), turned to -90 degrees
- moved R13 65.8 mm to (97.0, 65.0), turned to 180 degrees
- moved J1 64.7 mm to (175.5, 43.0)
- moved J5 63.5 mm to (181.2, 45.5), turned to 180 degrees
- moved R11 63.3 mm to (101.4, 71.0), turned to -90 degrees
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Connections:
- A1 pad 25: unconnected-(A1-A6-Pad25) -> Relay1
- A1 pad 26: unconnected-(A1-A7-Pad26) -> Relay2
- K1 pad 1: unconnected-(K1-+-Pad1) -> +5V
- K1 pad 8: COM -> Net-(K1--)
- K2 pad 1: unconnected-(K2-+-Pad1) -> +5V
- K2 pad 8: COM -> Net-(K2--)
- R10 pad 1: D11 -> D9
- R16 pad 1: D9 -> D11
- R19 pad 1: D8 -> D12
- R7 pad 1: D12 -> D8
- SW1 pad 1: NEXT -> PREVIOUS
- SW2 pad 1: PREVIOUS -> NEXT
Routing:
- net +5V: track 44.9 -> 294.2 mm, vias 1 -> 13
- net RESISTANCE: track 0.00 -> 148.6 mm, vias 0 -> 1
- net NEXT: track 0.00 -> 101.1 mm, vias 0 -> 1
- net BATTERY VOLTAGE: track 0.00 -> 99.3 mm, vias 0 -> 2
- net Relay1: track 0.00 -> 79.7 mm, vias 0 -> 1
- net RangeSel: track 9.31 -> 86.5 mm, vias 0 -> 2
- net Relay2: track 0.00 -> 68.0 mm, vias 0 -> 6
- net D5: track 0.00 -> 59.0 mm, vias 0 -> 1
- net PREVIOUS: track 0.00 -> 57.2 mm
- net VOLTAGE: track 0.00 -> 57.1 mm, vias 0 -> 2
- net FREQUENCY IN: track 0.00 -> 53.9 mm
- net CURRENT: track 0.00 -> 44.0 mm, vias 0 -> 2
- net D12: track 0.00 -> 29.9 mm
- net D11: track 0.00 -> 24.5 mm
- net Net-(U2-BW_SEL): track 0.00 -> 20.5 mm, vias 0 -> 2
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- added copper zone on B.Cu, net A
- added copper zone on F.Cu, net A
- added copper zone on B.Cu, net COM
- added copper zone on F.Cu, net COM
- added copper zone on B.Cu, net VRf
- added copper zone on F.Cu, net VRf

Commit message: Fixed minor issues
- Moved the relay further away from the current sensor.
- Added vias near the ground connection of the current sensort
- Swapped 3D models for the correct ones
- Moved ground plane away from the mounting holes
- Fixed pin capability related issue
Parts:
- moved K3 14.5 mm to (159.0, 99.0), turned to 90 degrees
Connections:
- A1 pad 19: RESISTANCE -> Relay1
- A1 pad 20: VOLTAGE -> Relay2
- A1 pad 25: Relay1 -> RESISTANCE
- A1 pad 26: Relay2 -> VOLTAGE
Routing:
- net Relay2: track 68.0 -> 85.5 mm, vias 6 -> 7
- net +5V: track 294.2 -> 308.5 mm, vias 13 -> 16
- net Relay1: track 79.7 -> 91.9 mm, vias 1 -> 3
- net VOLTAGE: track 57.1 -> 45.6 mm
- net HighRange: track 38.5 -> 49.7 mm
- net LowRange: track 25.8 -> 35.7 mm, vias 0 -> 2
- net NEXT: track 101.1 -> 104.7 mm
- net Net-(K3--): track 3.90 -> 7.03 mm, vias 0 -> 1
- net COM: track 6.11 -> 8.00 mm, vias 53 -> 59
- net RESISTANCE: track 148.6 -> 147.6 mm, vias 1 -> 2
- net RangeSel: track 86.5 -> 87.3 mm
- net FREQUENCY IN: track 53.9 -> 53.2 mm

Commit message: V1.0 Complete
Parts:
- added C15: 0.1uF, Capacitor_SMD:C_0805_2012Metric_Pad1.18x1.45mm_HandSolder, F.Cu at (135.5, 68.5)
- added C16: 10nF, Capacitor_SMD:C_0805_2012Metric_Pad1.18x1.45mm_HandSolder, F.Cu at (122.5, 68.5)
- added J6: Conn_01x04_Pin, Connector_JST:JST_XH_B4B-XH-AM_1x04_P2.50mm_Vertical, F.Cu at (92.0, 121.8)
- added R32: 10k, Resistor_SMD:R_0805_2012Metric_Pad1.20x1.40mm_HandSolder, F.Cu at (179.0, 114.5)
- added R33: 150, Resistor_SMD:R_0805_2012Metric_Pad1.20x1.40mm_HandSolder, F.Cu at (177.0, 122.5)
- added R34: 10k, Resistor_SMD:R_0805_2012Metric_Pad1.20x1.40mm_HandSolder, F.Cu at (179.5, 98.0)
- added R35: 150, Resistor_SMD:R_0805_2012Metric_Pad1.20x1.40mm_HandSolder, F.Cu at (175.0, 99.0)
- added U6: LM35-D, Package_SO:SOIC-8_3.9x4.9mm_P1.27mm, F.Cu at (129.0, 70.5)
- J1, J5: footprint Connector_PinSocket_2.54mm:PinSocket_1x02_P2.54mm_Vertical -> Connector_JST:JST_XH_B2B-XH-AM_1x02_P2.50mm_Vertical
- moved D1 5.27 mm to (146.9, 113.5), turned to 0 degrees
- moved D2 5.00 mm to (160.0, 83.5), turned to 180 degrees
- moved R24 4.73 mm to (147.0, 118.0)
- moved C5 4.58 mm to (112.7, 73.5), turned to 90 degrees
- moved J1 1.41 mm to (174.5, 42.0), turned to -90 degrees
- moved J5 1.23 mm to (180.5, 44.5), turned to 90 degrees
- moved Q1 0.84 mm to (105.2, 76.0)
- moved Q2 0.84 mm to (105.2, 71.0)
- moved Q3 0.84 mm to (105.2, 66.0)
- moved Q4 0.84 mm to (105.2, 61.0)
- moved Q5 0.84 mm to (105.2, 56.0)
- moved R10 0.84 mm to (96.1, 70.0)
- moved R11 0.84 mm to (100.6, 71.0)
- moved R12 0.84 mm to (109.6, 71.0)
- moved R13 0.84 mm to (96.2, 65.0)
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Connections:
- A1 pad 10: unconnected-(A1-D7-Pad10) -> Relay2
- A1 pad 20: Relay2 -> TEMPERATURE
- Q7 pad 2: Relay1 -> Net-(Q7-G)
- Q8 pad 2: Relay2 -> Net-(Q8-G)
Routing:
- net +5V: track 308.5 -> 363.2 mm, vias 16 -> 18
- net TEMPERATURE: track 0.00 -> 44.8 mm, vias 0 -> 2
- net SCL: track 0.00 -> 30.6 mm, vias 0 -> 3
- net SDA: track 0.00 -> 30.3 mm, vias 0 -> 3
- net Net-(Q7-G): track 0.00 -> 7.41 mm
- net Net-(Q8-G): track 0.00 -> 7.17 mm
- net Net-(D2-K): track 11.4 -> 16.4 mm
- net HighRange: track 49.7 -> 44.9 mm, vias 3 -> 2
- net Net-(D1-K): track 9.45 -> 6.49 mm
- net Relay1: track 91.9 -> 89.0 mm
- net VOLTAGE IN: track 18.3 -> 16.3 mm
- net Relay2: track 85.5 -> 87.3 mm, vias 7 -> 6
- net +9V: track 16.1 -> 17.5 mm
- net Net-(J5-Pin_1): track 16.2 -> 15.5 mm
- net D5: track 59.0 -> 59.7 mm
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Other:
- board text added: "BAT"
- board text added: "BT"
- board text added: "CURRENT"
- board text added: "DJ"
- board text added: "FREQUENCY"
- board text added: "GND SCL SDA +5V"
- board text added: "LCD"
- board text added: "MS"
- board text added: "RELAY MATRIX"
- board text added: "RESISTANCE"
- board text added: "SPROJ 1 Group 5 MS, TEDH, BT, DJ V1.0"
- board text added: "SWITCH"
- board text added: "TEDH"
- board text added: "TEMPERATURE"
- board text added: "VOLTAGE"
